File: Keyboard PCB STM32.kicad_pcb (KiCad board)
At the start: 2 copper layers, 309.8 x 101.8 mm, 156 parts, among them J1 USB_C_Receptacle_USB2.0_14P, SW1 1u, SW10 1u, SW11 1u, SW12 1u, SW13 1u, SW14 2u, SW15 1u, SW16 1.5u, SW17 1u, SW18 1u, SW19 1u, SW2 1u, SW20 1u, SW21 1u, SW22 1u, SW23 1u, SW24 1u, SW25 1u, SW26 1u, SW27 1u, SW28 1u, SW29 1.5u, SW3 1u, SW30 1u, SW31 1.75u, SW32 1u, SW33 1u, SW34 1u, SW35 1u, SW36 1u, SW37 1u, SW38 1u, SW39 1u, SW4 1u, SW40 1u, SW41 1u, SW42 1u, SW43 2.25u, SW44 1u, SW45 2.25u, SW46 1u, SW47 1u, SW48 1u, SW49 1u, SW5 1u, SW50 1u, SW51 1u, SW52 1u, SW53 1u, SW54 1u, SW55 1u, SW56 1.75u, SW57 1u, SW58 1u, SW59 1.25u, SW6 1u, SW60 1.25u, SW61 1.25u, SW62 6.25u, SW63 1.25u, SW64 1.25u, SW65 1u, SW66 1u, SW67 1u, SW68 SW_Push, SW7 1u, SW8 1u, SW9 1u, U1 XC6206PxxxMR, U2 SRV05-4, U3 STM32F072CBTx

Commit message: Update to ESD protection
Changed ESD from SRV05-4 to USBLC6-2SC6
Parts:
- U2: value SRV05-4 -> USBLC6-2SC6

Commit message: Add files via upload
Parts:
- added SW69: SW_Push, Button_Switch_SMD:SW_Push_1P1T_XKB_TS-1187A, B.Cu at (176.6, 117.5)
- SW68: footprint Button_Switch_SMD:SW_SPST_TS-1088-xR020 -> Button_Switch_SMD:Panasonic_EVQPUL_EVQPUC
- moved R3 9.00 mm to (202.2, 117.7), turned to -90 degrees
- moved SW68 1.11 mm to (196.8, 117.7), turned to 0 degrees
Routing:
- net BOOT: track 15.6 -> 36.7 mm
- net +3.3V: track 87.3 -> 100.7 mm
- net R4: track 458.9 -> 461.3 mm
